File: kicad/8led2.sch (KiCad schematic (older format))
At the start: 27 parts, among them J1 PMOD, J2 PMOD

Commit message: update schema, add BOM
Other:
- note added: "JP1 can be used to accomodate\ncommon-anode LED types."
- moved on the sheet: D1, D2, D3, D4, D5, D6, D7, D8, J1, J2, JP1, R1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
